File: hardware/kicad/24S-DCDC.kicad_pcb (KiCad board)
At the start: 2 copper layers, 100 x 100 mm, 11 parts, among them J1 J1, J2_48V J2_48V, J3_12V J3_12V, J4_5V J4_5V

Commit message: Add files via upload
Routing:
- net GND: track 82.5 -> 75.5 mm
Other:
- board text added: "24S-DCDC v0.8 pre-route — NOT FOR FAB"
Changed lines of the file:
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@@
   (net 5 "V5")
   (gr_rect (start 0 0) (end 100 100) (layer "Edge.Cuts") (width 0.1))
+  (gr_text "24S-DCDC v0.8 pre-route — NOT FOR FAB" (at 50 5) (layer "F.SilkS") (effects (font (size 1.2 1.2) (thickness 0.18))))
   (footprint "MountHole:M3" (layer "F.Cu") (at 4 4) (attr board_only exclude_from_bom exclude_from_pos_files)
     (fp_text reference "MH1" (at 0 -3) (layer "F.SilkS") (effects (font (size 1 1) (thickness 0.15))))
@@
   (segment (start 17.5 50) (end 50 50) (width 2.0) (layer "F.Cu") (net 2))
   (segment (start 50 50) (end 50 68) (width 2.0) (layer "F.Cu") (net 2))
-  (segment (start 50 50) (end 50 43) (width 2.0) (layer "F.Cu") (net 2))
   (segment (start 50 43) (end 50 18) (width 2.0) (layer "F.Cu") (net 2))
   (segment (start 60 75) (end 90 75) (width 2.0) (layer "F.Cu") (net 3))
